File: safewise.kicad_pcb (KiCad board)
At the start: 2 copper layers, 32.1 x 37.5 mm, 44 parts, among them IC1 MCP1700T-3002E/TT, K1 USB_OTG, K2 TC2030-JTAG, SW1 SW_DIP_x01, SW2 SW_DIP_x01, U1 STM32F205RETx, U3 UG-2864HSWEG01, Y1 8MHz

Commit message: SafeWISE pcb version 1.1
Parts:
- K1: footprint micorusb:USB_Micro_B-10118194-0001LF_handsoldering -> micorusb:USB_Micro_B-10118194-0001LF_handsoldering_pads
- moved R7 0.72 mm to (154.1, 120.1)
Routing:
- net Net-(D1-Pad4): track 24.3 -> 25.0 mm
Other:
- board text added: "COINWISE SAFEWISE v1.1"
- board text removed: "COINWISE TREASURE v1.0"

Commit message: SafeWISE pcb version 1.2
Parts:
- moved U3 1.78 mm to (158.7, 93.5)
Routing:
- net GND: track 216.5 -> 211.8 mm, vias 17 -> 18
- net +3V3: track 121.1 -> 124.4 mm
- net Net-(U1-Pad23): track 19.6 -> 21.4 mm
- net Net-(U1-Pad20): track 25.1 -> 26.9 mm
- net Net-(U1-Pad26): track 16.0 -> 17.8 mm
- net Net-(C18-Pad1): track 9.52 -> 11.3 mm
- net Net-(U1-Pad27): track 15.9 -> 17.7 mm
- net Net-(U1-Pad21): track 17.8 -> 19.6 mm
- net Net-(C5-Pad2): track 3.15 -> 4.93 mm
- net Net-(C4-Pad2): track 3.28 -> 5.06 mm
- net Net-(C4-Pad1): track 3.32 -> 5.10 mm
- net Net-(R10-Pad2): track 3.96 -> 5.39 mm
- net Net-(C18-Pad2): track 4.90 -> 5.74 mm
- net SWDIO: track 44.1 -> 44.7 mm
Other:
- board text added: "COINWISE SAFEWISE v1.2"
- board text removed: "COINWISE SAFEWISE v1.1"
